File: DCDC.kicad_sch (KiCad schematic)
At the start: 6 parts, among them J1 XT60, J2 XT60, Q5 Q_NMOS_GDS, Q6 Q_NMOS_GDS

Commit message: Autosave
Connections:
- net Vin_DCDC_shunt is gone; now on net VinDCDC: Q5.2 (D), Q6.2 (D)
Changed lines of the file:
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@@
 		)
 	)
-	(hierarchical_label "Vin_DCDC_cap"
+	(hierarchical_label "Vin_DCDC_shunt"
 		(shape output)
 		(at 67.31 26.67 0)

Commit message: Autosave
Connections:
- net VinDCDC: no longer Q5.2 (D), Q6.2 (D)
- new net Gatedriver/Vs_node: Q5.2 (D), Q6.2 (D)
Changed lines of the file:
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@@
 	(wire
 		(pts
-			(xy 66.04 26.67) (xy 67.31 26.67)
+			(xy 66.04 27.94) (xy 67.31 27.94)
 		)
 		(stroke
@@
 	(wire
 		(pts
-			(xy 66.04 26.67) (xy 66.04 25.4)
+			(xy 66.04 27.94) (xy 66.04 25.4)
 		)
 		(stroke
@@
 		)
 	)
-	(label "Vin_DCDC_shunt"
-		(at 76.2 25.4 0)
-		(effects
-			(font
-				(size 1.27 1.27)
-			)
-			(justify left bottom)
-		)
-	)
 	(label "Hin"
 		(at 114.3 43.18 0)
@@
 	(hierarchical_label "Vin_DCDC_shunt"
 		(shape output)
-		(at 67.31 26.67 0)
+		(at 67.31 27.94 0)
 		(effects
 			(font

Commit message: Autosave
Connections:
- net Gatedriver/Vs_node is gone; now on net VinDCDC: Q5.2 (D), Q6.2 (D)
Changed lines of the file:
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@@
 		)
 	)
-	(hierarchical_label "Vin_DCDC_shunt"
+	(hierarchical_label "Vin_DCDC_shunt_input side"
 		(shape output)
 		(at 67.31 27.94 0)
 		(effects
 			(font
+				(size 1.27 1.27)
+			)
+			(justify left)
+		)
+	)
+	(hierarchical_label "Vin_DCDC_shunt_input side"
+		(shape output)
+		(at 76.2 25.4 0)
+		(effects
+			(font

Commit message: Autosave
Connections:
- net VinDCDC: no longer Q5.2 (D), Q6.2 (D)
- new net Vin_DCDC_shunt_output_side: Q5.2 (D), Q6.2 (D)
Changed lines of the file:
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@@
 		)
 	)
-	(hierarchical_label "Vin_DCDC_shunt_input side"
-		(shape output)
+	(hierarchical_label "Vin_DCDC_shunt_output_side"
+		(shape input)
 		(at 76.2 25.4 0)
 		(effects
