File: DCDC.kicad_sch (KiCad schematic)
At the start: 5 parts, among them J1 XT60, Q5 Q_NMOS_GDS, Q6 Q_NMOS_GDS

Commit message: Autosave
Connections:
- net VinDCDC: no longer Q5.2 (D), Q6.2 (D)
- net Vin_DCDC_coil_source_side: now reaches J1.2 (Pin_2)
- new net Vin_DCDC_shunt_output_side: Q5.2 (D), Q6.2 (D)
Changed lines of the file:
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@@
-		)
-	)
-	(hierarchical_label "Vin_DCDC_shunt_output_side"
-		(shape input)
-		(at 45.72 25.4 90)
-		(effects
-			(font
-				(size 1.27 1.27)
-			)
-			(justify left)
 		)
 	)
@@
 		(effects
 			(font
+				(size 1.27 1.27)
+			)
+			(justify left)
+		)
+	)
+	(hierarchical_label "Vin_DCDC_coil_source_side"
+		(shape input)
+		(at 41.91 25.4 90)
+		(effects
+			(font

Commit message: Autosave
Connections:
- net Vin_DCDC_coil_source_side is gone; now on net VinDCDC: J1.2 (Pin_2)
Changed lines of the file:
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@@
+		)
+	)
+	(hierarchical_label "Vin_DCDC_coil_source_side"
+		(shape output)
+		(at 45.72 25.4 90)
+		(effects
+			(font
+				(size 1.27 1.27)
+			)
+			(justify left)
 		)
 	)
@@
 	)
 	(hierarchical_label "Vin_DCDC_coil_source_side"
-		(shape input)
+		(shape output)
 		(at 41.91 25.4 90)
 		(effects

Commit message: Autosave
Connections:
- net VinDCDC: no longer J1.2 (Pin_2)
- new net Vin_DCDC_coil_source_side: J1.2 (Pin_2)
Changed lines of the file:
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@@
 		)
 	)
-	(hierarchical_label "Vin_DCDC_coil_source_side"
-		(shape output)
+	(hierarchical_label "Vin_DCDC_coil_circuit_side"
+		(shape input)
 		(at 45.72 25.4 90)
 		(effects

Commit message: Autosave
Parts:
- removed J1: XT60, symbol Connector:Screw_Terminal_01x02
Changed lines of the file:
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@@
 		)
 	)
-	(hierarchical_label "Vin_DCDC_coil_source_side"
+	(hierarchical_label "Vin_DCDC_coil_input_side"
 		(shape output)
 		(at 41.91 25.4 90)
@@
 					(unit 1)
 				)
-			)
-		)
-	)
-	(symbol
-		(lib_id "Connector:Screw_Terminal_01x02")
-		(at 30.48 39.37 180)
-		(unit 1)
-		(body_style 1)
-		(exclude_from_sim no)
-		(in_bom yes)
-		(on_board yes)
-		(in_pos_files yes)
-		(dnp no)
-		(fields_autoplaced yes)
-		(property "Reference" "J1"
-			(at 30.48 30.48 0)
-			(show_name no)
-			(do_not_autoplace no)
-			(effects
-				(font
-					(size 1.27 1.27)
-				)
-			)
-		)
-		(property "Value" "XT60"
-			(at 30.48 33.02 0)
-			(show_name no)
-			(do_not_autoplace no)
-			(effects
-				(font
-					(size 1.27 1.27)
-				)
-			)
-		)
-		(property "Footprint" ""
-			(at 30.48 39.37 0)
-			(hide yes)
-			(show_name no)
-			(do_not_autoplace no)
-			(effects
-				(font
-					(size 1.27 1.27)
-				)
-			)
-		)
-		(property "Datasheet" ""
-			(at 30.48 39.37 0)
-			(hide yes)
-			(show_name no)
-			(do_not_autoplace no)
-			(effects
-				(font
-					(size 1.27 1.27)
-				)
-			)
-		)
-		(property "Description" "Generic screw terminal, single row, 01x02, script generated (kicad-library-utils/schlib/autogen/connector/)"
-			(at 30.48 39.37 0)
-			(hide yes)
-			(show_name no)
-			(do_not_autoplace no)
-			(effects
-				(font
-					(size 1.27 1.27)
-				)
-			)
-		)
-		(pin "1"
-		)
-		(pin "2"
-		)
-		(instances
-			(project "WET_PCB_v2"
-				(path "/13451c35-1666-47d9-9525-8d8125ba1cf3/04007180-46fe-4cf0-9e6f-a7d321798318"
-					(reference "J1")
-					(unit 1)
-				)

Commit message: Autosave
Connections:
- net GND: no longer names the net of C11.2, C12.2, Q5.3 (S)
- net VinDCDC renamed Vin_DCDC_coil_circuit_side
Changed lines of the file:
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@@
-	)
-	(junction
-		(at 52.07 25.4)
-		(diameter 0)
-		(color 0 0 0 0)
 	)
 	(junction
@@
 	)
 	(junction
-		(at 52.07 50.8)
-		(diameter 0)
-		(color 0 0 0 0)
-	)
-	(junction
 		(at 100.33 25.4)
 		(diameter 0)
@@
 	(wire
 		(pts
-			(xy 52.07 50.8) (xy 86.36 50.8)
-		)
-		(stroke
-			(width 0)
-			(type default)
-		)
-	)
-	(wire
-		(pts
 			(xy 93.98 45.72) (xy 93.98 41.91)
 		)
@@
 	(wire
 		(pts
-			(xy 49.53 50.8) (xy 52.07 50.8)
+			(xy 49.53 50.8) (xy 86.36 50.8)
 		)
 		(stroke
@@
 	(wire
 		(pts
-			(xy 49.53 25.4) (xy 52.07 25.4)
+			(xy 49.53 25.4) (xy 67.31 25.4)
 		)
 		(stroke
@@
 		(pts
 			(xy 170.18 41.91) (xy 170.18 50.8)
-		)
-		(stroke
-			(width 0)
-			(type default)
-		)
-	)
-	(wire
-		(pts
-			(xy 52.07 25.4) (xy 67.31 25.4)
 		)
 		(stroke
@@
 					(unit 1)
 				)
-			)
-		)
-	)
-	(symbol
-		(lib_id "power:VCC")
-		(at 52.07 25.4 0)
-		(unit 1)
-		(body_style 1)
-		(exclude_from_sim no)
-		(in_bom yes)
-		(on_board yes)
-		(in_pos_files yes)
-		(dnp no)
-		(fields_autoplaced yes)
-		(property "Reference" "#PWR013"
-			(at 52.07 29.21 0)
-			(hide yes)
-			(show_name no)
-			(do_not_autoplace no)
-			(effects
-				(font
-					(size 1.27 1.27)
-				)
-			)
-		)
-		(property "Value" "VinDCDC"
-			(at 52.07 20.32 0)
-			(show_name no)
-			(do_not_autoplace no)
-			(effects
-				(font
-					(size 1.27 1.27)
-				)
-			)
-		)
-		(property "Footprint" ""
-			(at 52.07 25.4 0)
-			(hide yes)
-			(show_name no)
-			(do_not_autoplace no)
-			(effects
-				(font
-					(size 1.27 1.27)
-				)
-			)
-		)
-		(property "Datasheet" ""
-			(at 52.07 25.4 0)
-			(hide yes)
-			(show_name no)
-			(do_not_autoplace no)
-			(effects
-				(font
-					(size 1.27 1.27)
-				)
-			)
-		)
-		(property "Description" "Power symbol creates a global label with name \"VCC\""
-			(at 52.07 25.4 0)
-			(hide yes)
-			(show_name no)
-			(do_not_autoplace no)
-			(effects
-				(font
-					(size 1.27 1.27)
-				)
-			)
-		)
-		(pin "1"
-		)
-		(instances
-			(project "WET_PCB_v2"
-				(path "/13451c35-1666-47d9-9525-8d8125ba1cf3/04007180-46fe-4cf0-9e6f-a7d321798318"
-					(reference "#PWR013")
-					(unit 1)
-				)
-			)
-		)
-	)
-	(symbol
-		(lib_id "power:GND")
-		(at 52.07 50.8 0)
-		(unit 1)
-		(body_style 1)
-		(exclude_from_sim no)
-		(in_bom yes)
-		(on_board yes)
-		(in_pos_files yes)
-		(dnp no)
-		(fields_autoplaced yes)
-		(property "Reference" "#PWR014"
-			(at 52.07 57.15 0)
-			(hide yes)
-			(show_name no)
-			(do_not_autoplace no)
-			(effects
-				(font
-					(size 1.27 1.27)
-				)
-			)
-		)
-		(property "Value" "GND"
-			(at 52.07 55.88 0)
-			(show_name no)
-			(do_not_autoplace no)
-			(effects
-				(font
-					(size 1.27 1.27)
-				)
-			)
-		)
-		(property "Footprint" ""
-			(at 52.07 50.8 0)
-			(hide yes)
-			(show_name no)
-			(do_not_autoplace no)
-			(effects
-				(font
-					(size 1.27 1.27)
-				)
-			)
-		)
-		(property "Datasheet" ""
-			(at 52.07 50.8 0)
-			(hide yes)
-			(show_name no)
-			(do_not_autoplace no)
-			(effects
-				(font
-					(size 1.27 1.27)
-				)
-			)
-		)
-		(property "Description" "Power symbol creates a global label with name \"GND\" , ground"
-			(at 52.07 50.8 0)
-			(hide yes)
-			(show_name no)
-			(do_not_autoplace no)
-			(effects
-				(font
-					(size 1.27 1.27)
-				)
-			)
-		)
-		(pin "1"
-		)
-		(instances
-			(project "WET_PCB_v2"
-				(path "/13451c35-1666-47d9-9525-8d8125ba1cf3/04007180-46fe-4cf0-9e6f-a7d321798318"
-					(reference "#PWR014")
-					(unit 1)
-				)
