File: DCDC.kicad_sch (KiCad schematic)
At the start: 4 parts, among them Q5 Q_NMOS_GDS, Q6 Q_NMOS_GDS

Commit message: Autosave
Connections:
- net Vin_DCDC_coil_circuit_side renamed DCDC_coil_circuit_side
Changed lines of the file:
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@@
 		)
 	)
-	(hierarchical_label "Vin_DCDC_coil_circuit_side"
+	(hierarchical_label "DCDC_coil_circuit_side"
 		(shape input)
 		(at 50.8 43.18 90)
@@
 		)
 	)
-	(hierarchical_label "Vin_DCDC_coil_input_side"
+	(hierarchical_label "DCDC_coil_input_side"
 		(shape output)
 		(at 44.45 43.18 90)

Commit message: SCH Save: 1 files changed DCDC.kicad_sch 0/0/2
Connections:
- net DCDC_coil_circuit_side renamed Vin_DCDC_coil_circuit_side
Changed lines of the file:
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@@
 		)
 	)
-	(hierarchical_label "DCDC_coil_circuit_side"
+	(hierarchical_label "Vin_DCDC_coil_circuit_side"
 		(shape input)
 		(at 50.8 43.18 90)
@@
 		)
 	)
-	(hierarchical_label "DCDC_coil_input_side"
+	(hierarchical_label "Vin_DCDC_coil_input_side"
 		(shape output)
 		(at 44.45 43.18 90)

Commit message: SCH Save: 1 files changed DCDC.kicad_sch 10/0/3
Connections:
- net Vin_DCDC_coil_circuit_side renamed DCDC_coil_circuit_side
Other:
- note added: "is one cap at in and out enough or do we want to add more (we can leave them empty anyway)"
Changed lines of the file:
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@@
 	(generator_version "10.0")
 	(paper "A4")
+	(text "is one cap at in and out enough or do we want to add more (we can leave them empty anyway)"
+		(exclude_from_sim no)
+		(at 116.078 75.692 0)
+		(effects
+			(font
+				(size 1.27 1.27)
+			)
+		)
+	)
 	(junction
 		(at 54.61 43.18)
@@
 		)
 	)
-	(hierarchical_label "Vin_DCDC_coil_circuit_side"
+	(hierarchical_label "DCDC_coil_circuit_side"
 		(shape input)
 		(at 50.8 43.18 90)
@@
 		)
 	)
-	(hierarchical_label "Vin_DCDC_coil_input_side"
+	(hierarchical_label "DCDC_coil_input_side"
 		(shape output)
 		(at 44.45 43.18 90)
