File: GateDriver.kicad_sch (KiCad schematic)
At the start: 11 parts, among them U4 IR2110

Commit message: Autosave
Connections:
- net VCC_Driver renamed VCC_Driver_DCDC
- net VDD_Driver renamed VDD_Driver_DCDC
Changed lines of the file:
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@@
 		)
 	)
-	(hierarchical_label "VDD_Driver"
+	(hierarchical_label "VDD_Driver_DCDC"
 		(shape input)
 		(at 82.55 24.13 90)
@@
 		)
 	)
-	(hierarchical_label "VCC_Driver"
+	(hierarchical_label "VCC_Driver_DCDC"
 		(shape input)
 		(at 92.71 24.13 90)

Commit message: SCH Save: 2 files changed GateDriver.kicad_sch 0/0/2 inverter.kicad_sch 0/0/2
Connections:
- net VCC_Driver_DCDC renamed VCC_Driver
- net VDD_Driver_DCDC renamed VDD_Driver
Changed lines of the file:
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@@
 		)
 	)
-	(hierarchical_label "VDD_Driver_DCDC"
+	(hierarchical_label "VDD_Driver"
 		(shape input)
 		(at 82.55 24.13 90)
@@
 		)
 	)
-	(hierarchical_label "VCC_Driver_DCDC"
+	(hierarchical_label "VCC_Driver"
 		(shape input)
 		(at 92.71 24.13 90)

Commit message: Autosave
Other:
- note added: "Add decoupling caps for VSS VDD"
Changed lines of the file:
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@@
 	(generator_version "10.0")
 	(paper "A4")
+	(text "Add decoupling caps for VSS VDD"
+		(exclude_from_sim no)
+		(at 61.468 80.264 0)
+		(effects
+			(font
+				(size 1.27 1.27)
+			)
+		)
+	)
 	(text "HIn = the input high from the MCU\nLin = PWM low from the mcu\nSD = shutdown tie to +12V"
 		(exclude_from_sim no)

Commit message: Autosave
Other:
- note removed: "Add decoupling caps for VSS VDD"
Changed lines of the file:
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@@
 	(generator_version "10.0")
 	(paper "A4")
-	(text "Add decoupling caps for VSS VDD"
-		(exclude_from_sim no)
-		(at 61.468 80.264 0)
-		(effects
-			(font
-				(size 1.27 1.27)
-			)
-		)
-	)
 	(text "HIn = the input high from the MCU\nLin = PWM low from the mcu\nSD = shutdown tie to +12V"
 		(exclude_from_sim no)
