File: inverter.kicad_sch (KiCad schematic)
At the start: 28 parts, among them Q1 IRF530NPBF, Q2 IRF530NPBF, Q3 IRF530NPBF, Q4 IRF530NPBF, U1 IR2110, U2 IR2110

Commit message: Autosave
Connections:
- net Inv_Driver_Left_Hin: now also U2.10 (HIN)
Changed lines of the file:
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@@
 	(hierarchical_label "Inv_Driver_Left_Hin"
 		(shape input)
-		(at 256.54 59.69 270)
+		(at 257.81 59.69 0)
 		(effects
 			(font
 				(size 1.27 1.27)
 			)
-			(justify right)
+			(justify left)
 		)
 	)

Commit message: Autosave
Connections:
- net Inv_Driver_Left_Hin: no longer U2.10 (HIN)
- net Inv_Driver_Right_Hin: now reaches U2.12 (LIN)
- net Inv_Driver_Right_Hin: now also U2.10 (HIN)
Changed lines of the file:
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@@
+		)
+	)
+	(hierarchical_label "Inv_Driver_Right_Hin"
+		(shape input)
+		(at 257.81 62.23 0)
+		(effects
+			(font
+				(size 1.27 1.27)
+			)
+			(justify left)
 		)
 	)
@@
 		)
 	)
-	(hierarchical_label "Inv_Driver_Left_Hin"
+	(hierarchical_label "Inv_Driver_Right_Hin"
 		(shape input)
 		(at 257.81 59.69 0)

Commit message: Autosave
Connections:
- net Inv_Driver_Right_Hin: no longer U2.12 (LIN)
- new net Inv_Driver_Right_LHin: U2.12 (LIN)
Changed lines of the file:
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@@
 		)
 	)
-	(hierarchical_label "Inv_Driver_Right_Hin"
+	(hierarchical_label "Inv_Driver_Right_LHin"
 		(shape input)
 		(at 257.81 62.23 0)

Commit message: Autosave
Connections:
- net Inv_Driver_Right_LHin is gone; now on net Inv_Driver_Right_Lin: U2.12 (LIN)
- net Inv_Driver_Right_Lin: now reaches U2.11 (SD)
Changed lines of the file:
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@@
 		)
 	)
-	(hierarchical_label "Inv_Driver_Right_LHin"
+	(hierarchical_label "Inv_Driver_Right_Lin"
 		(shape input)
 		(at 257.81 62.23 0)
@@
 		(effects
 			(font
+				(size 1.27 1.27)
+			)
+			(justify left)
+		)
+	)
+	(hierarchical_label "Inv_Driver_Right_Lin"
+		(shape input)
+		(at 257.81 64.77 0)
+		(effects
+			(font

Commit message: Autosave
Connections:
- net Inv_Driver_Right_Lin: no longer U2.11 (SD)
- new net Inv_Driver_Right_SD: U2.11 (SD)
Changed lines of the file:
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@@
 		)
 	)
-	(hierarchical_label "Inv_Driver_Right_Lin"
+	(hierarchical_label "Inv_Driver_Right_SD"
 		(shape input)
 		(at 257.81 64.77 0)

Commit message: Autosave
Connections:
- net 12V: no longer U1.3 (VCC)
- new net VCC_Inverter: U1.3 (VCC)
Changed lines of the file:
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@@
+		)
+	)
+	(label "VCC_Inverter"
+		(at 55.88 64.77 0)
+		(effects
+			(font
+				(size 1.27 1.27)
+			)
+			(justify left bottom)
 		)
 	)
@@
 					(unit 1)
 				)
-			)
-		)
-	)
-	(symbol
-		(lib_id "power:VCC")
-		(at 55.88 64.77 270)
-		(unit 1)
-		(body_style 1)
-		(exclude_from_sim no)
-		(in_bom yes)
-		(on_board yes)
-		(in_pos_files yes)
-		(dnp no)
-		(fields_autoplaced yes)
-		(property "Reference" "#PWR06"
-			(at 52.07 64.77 0)
-			(hide yes)
-			(show_name no)
-			(do_not_autoplace no)
-			(effects
-				(font
-					(size 1.27 1.27)
-				)
-			)
-		)
-		(property "Value" "12V"
-			(at 59.69 64.7699 90)
-			(show_name no)
-			(do_not_autoplace no)
-			(effects
-				(font
-					(size 1.27 1.27)
-				)
-				(justify left)
-			)
-		)
-		(property "Footprint" ""
-			(at 55.88 64.77 0)
-			(hide yes)
-			(show_name no)
-			(do_not_autoplace no)
-			(effects
-				(font
-					(size 1.27 1.27)
-				)
-			)
-		)
-		(property "Datasheet" ""
-			(at 55.88 64.77 0)
-			(hide yes)
-			(show_name no)
-			(do_not_autoplace no)
-			(effects
-				(font
-					(size 1.27 1.27)
-				)
-			)
-		)
-		(property "Description" "Power symbol creates a global label with name \"VCC\""
-			(at 55.88 64.77 0)
-			(hide yes)
-			(show_name no)
-			(do_not_autoplace no)
-			(effects
-				(font
-					(size 1.27 1.27)
-				)
-			)
-		)
-		(pin "1"
-		)
-		(instances
-			(project "WET_PCB_v2"
-				(path "/13451c35-1666-47d9-9525-8d8125ba1cf3/a035cbd1-b4bf-441e-99d9-9f1401ee5bfe"
-					(reference "#PWR06")
-					(unit 1)
-				)

Commit message: Autosave
Connections:
- net 12V: no longer D1.2 (A)
- net 5V: no longer C1.2, U1.9 (VDD)
- net VCC_Inverter: now also D1.2 (A)
- new net: C1.2, U1.9 (VDD)
Changed lines of the file:
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@@
 		)
 	)
+	(label "VCC_Inverter"
+		(at 54.61 25.4 0)
+		(effects
+			(font
+				(size 1.27 1.27)
+			)
+			(justify left bottom)
+		)
+	)
 	(label "Vin"
 		(at 147.32 17.78 0)
@@
 	)
 	(symbol
-		(lib_id "power:VCC")
-		(at 54.61 25.4 0)
-		(unit 1)
-		(body_style 1)
-		(exclude_from_sim no)
-		(in_bom yes)
-		(on_board yes)
-		(in_pos_files yes)
-		(dnp no)
-		(fields_autoplaced yes)
-		(property "Reference" "#PWR04"
-			(at 54.61 29.21 0)
-			(hide yes)
-			(show_name no)
-			(do_not_autoplace no)
-			(effects
-				(font
-					(size 1.27 1.27)
-				)
-			)
-		)
-		(property "Value" "12V"
-			(at 54.61 20.32 0)
-			(show_name no)
-			(do_not_autoplace no)
-			(effects
-				(font
-					(size 1.27 1.27)
-				)
-			)
-		)
-		(property "Footprint" ""
-			(at 54.61 25.4 0)
-			(hide yes)
-			(show_name no)
-			(do_not_autoplace no)
-			(effects
-				(font
-					(size 1.27 1.27)
-				)
-			)
-		)
-		(property "Datasheet" ""
-			(at 54.61 25.4 0)
-			(hide yes)
-			(show_name no)
-			(do_not_autoplace no)
-			(effects
-				(font
-					(size 1.27 1.27)
-				)
-			)
-		)
-		(property "Description" "Power symbol creates a global label with name \"VCC\""
-			(at 54.61 25.4 0)
-			(hide yes)
-			(show_name no)
-			(do_not_autoplace no)
-			(effects
-				(font
-					(size 1.27 1.27)
-				)
-			)
-		)
-		(pin "1"
-		)
-		(instances
-			(project "WET_PCB_v2"
-				(path "/13451c35-1666-47d9-9525-8d8125ba1cf3/a035cbd1-b4bf-441e-99d9-9f1401ee5bfe"
-					(reference "#PWR04")
-					(unit 1)
-				)
-			)
-		)
-	)
-	(symbol
 		(lib_id "Device:C_Polarized")
 		(at 147.32 63.5 90)
@@
 					(unit 1)
 				)
-			)
-		)
-	)
-	(symbol
-		(lib_id "power:VCC")
-		(at 44.45 25.4 0)
-		(unit 1)
-		(body_style 1)
-		(exclude_from_sim no)
-		(in_bom yes)
-		(on_board yes)
-		(in_pos_files yes)
-		(dnp no)
-		(property "Reference" "#PWR05"
-			(at 44.45 29.21 0)
-			(hide yes)
-			(show_name no)
-			(do_not_autoplace no)
-			(effects
-				(font
-					(size 1.27 1.27)
-				)
-			)
-		)
-		(property "Value" "5V"
-			(at 44.958 20.32 0)
-			(show_name no)
-			(do_not_autoplace no)
-			(effects
-				(font
-					(size 1.27 1.27)
-				)
-			)
-		)
-		(property "Footprint" ""
-			(at 44.45 25.4 0)
-			(hide yes)
-			(show_name no)
-			(do_not_autoplace no)
-			(effects
-				(font
-					(size 1.27 1.27)
-				)
-			)
-		)
-		(property "Datasheet" ""
-			(at 44.45 25.4 0)
-			(hide yes)
-			(show_name no)
-			(do_not_autoplace no)
-			(effects
-				(font
-					(size 1.27 1.27)
-				)
-			)
-		)
-		(property "Description" "Power symbol creates a global label with name \"VCC\""
-			(at 44.45 25.4 0)
-			(hide yes)
-			(show_name no)
-			(do_not_autoplace no)
-			(effects
-				(font
-					(size 1.27 1.27)
-				)
-			)
-		)
-		(pin "1"
-		)
-		(instances
-			(project "WET_PCB_v2"
-				(path "/13451c35-1666-47d9-9525-8d8125ba1cf3/a035cbd1-b4bf-441e-99d9-9f1401ee5bfe"
-					(reference "#PWR05")
-					(unit 1)
-				)
