File: WET_PCB_v2.kicad_sch (KiCad schematic)
At the start: 24 parts, among them J10 Conn_01x09_Pin, J11 Conn_01x09_Pin, J2 Conn_01x09_Pin, J3 Conn_01x09_Pin, J4 XT60, J5 Barrel jack, J6 Pluggable Terminal Block, J7 Pluggable Terminal Block, J8 Jumper, U3 Opamp_Quad

Commit message: Autosave
Parts:
- C18: footprint (none) -> Capacitor_THT:CP_Radial_D5.0mm_P2.00mm
Changed lines of the file:
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@@
 			)
 		)
-		(property "Footprint" ""
+		(property "Footprint" "Capacitor_THT:CP_Radial_D5.0mm_P2.00mm"
 			(at 70.8152 88.9 0)
 			(hide yes)

Commit message: SCH Save: 1 files changed WET_PCB_v2.kicad_sch 0/0/2
Parts:
- R5, R6: footprint (none) -> Resistor_THT:R_Axial_DIN0207_L6.3mm_D2.5mm_P7.62mm_Horizontal
Changed lines of the file:
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@@
 			)
 		)
-		(property "Footprint" ""
+		(property "Footprint" "Resistor_THT:R_Axial_DIN0207_L6.3mm_D2.5mm_P7.62mm_Horizontal"
 			(at 18.542 80.01 90)
 			(hide yes)
@@
 			)
 		)
-		(property "Footprint" ""
+		(property "Footprint" "Resistor_THT:R_Axial_DIN0207_L6.3mm_D2.5mm_P7.62mm_Horizontal"
 			(at 29.972 80.01 90)
 			(hide yes)

Commit message: Autosave
Parts:
- C16, C17: footprint (none) -> Capacitor_THT:CP_Radial_D5.0mm_P2.00mm
Changed lines of the file:
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@@
 			)
 		)
-		(property "Footprint" ""
+		(property "Footprint" "Capacitor_THT:CP_Radial_D5.0mm_P2.00mm"
 			(at 58.1152 45.72 0)
 			(hide yes)
@@
 			)
 		)
-		(property "Footprint" ""
+		(property "Footprint" "Capacitor_THT:CP_Radial_D5.0mm_P2.00mm"
 			(at 40.3352 45.72 0)
 			(hide yes)

Commit message: SCH Save: 1 files changed WET_PCB_v2.kicad_sch 0/0/2
Parts:
- C20, C21: footprint (none) -> Capacitor_THT:CP_Radial_D5.0mm_P2.00mm
Changed lines of the file:
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@@
 			)
 		)
-		(property "Footprint" ""
+		(property "Footprint" "Capacitor_THT:CP_Radial_D5.0mm_P2.00mm"
 			(at 80.9752 67.31 0)
 			(hide yes)
@@
 			)
 		)
-		(property "Footprint" ""
+		(property "Footprint" "Capacitor_THT:CP_Radial_D5.0mm_P2.00mm"
 			(at 63.1952 67.31 0)
 			(hide yes)

Commit message: SCH Save: 1 files changed WET_PCB_v2.kicad_sch 10/0/0
Other:
- note added: "the caps have random footprints so they appear in the layout designer"
Changed lines of the file:
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@@
+		)
+	)
+	(text "the caps have random footprints \nso they appear in the layout designer"
+		(exclude_from_sim no)
+		(at 68.834 51.562 0)
+		(effects
+			(font
+				(size 1.27 1.27)
+			)
 		)
 	)

Commit message: SCH Save: 1 files changed WET_PCB_v2.kicad_sch 0/0/1
Parts:
- J7: footprint (none) -> Connector_Phoenix_GMSTB:PhoenixContact_GMSTBA_2,5_2-G-7,62_1x02_P7.62mm_Horizontal
Changed lines of the file:
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@@
 			)
 		)
-		(property "Footprint" ""
+		(property "Footprint" "Connector_Phoenix_GMSTB:PhoenixContact_GMSTBA_2,5_2-G-7,62_1x02_P7.62mm_Horizontal"
 			(at 245.11 26.67 0)
 			(hide yes)

Commit message: SCH Save: 1 files changed WET_PCB_v2.kicad_sch 10/0/0
Other:
- note added: "i did not add any testpoints we should check out where we need them"
Changed lines of the file:
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@@
+		)
+	)
+	(text "i did not add any testpoints we should check out where we need them"
+		(exclude_from_sim no)
+		(at 178.816 122.936 0)
+		(effects
+			(font
+				(size 1.27 1.27)
+			)
 		)
 	)

Commit message: most footprints added (some random)
Parts:
- J7: footprint Connector_Phoenix_GMSTB:PhoenixContact_GMSTBA_2,5_2-G-7,62_1x02_P7.62mm_Horizontal -> (none)
Other:
- note removed: "i did not add any testpoints we should check out where we need them"
Changed lines of the file:
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@@
-		)
-	)
-	(text "i did not add any testpoints we should check out where we need them"
-		(exclude_from_sim no)
-		(at 178.816 122.936 0)
-		(effects
-			(font
-				(size 1.27 1.27)
-			)
 		)
 	)
@@
 			)
 		)
-		(property "Footprint" "Connector_Phoenix_GMSTB:PhoenixContact_GMSTBA_2,5_2-G-7,62_1x02_P7.62mm_Horizontal"
+		(property "Footprint" ""
 			(at 245.11 26.67 0)
 			(hide yes)
