File: MCU.kicad_sch (KiCad schematic)
At the start: 0 parts

Commit message: Autosave
Parts:
- added C18, C19: C_Polarized, symbol Device:C_Polarized
- added J1: XT60, symbol Connector:Conn_01x02_Pin
- added U6: (no value), symbol WET:WET_Token_10
Connections:
- new net ADC1_IN0: U6.14 (EXT_ADC1_IN0)
- new net ADC1_IN1: U6.15 (EXT_ADC_IN1)
- new net ADC1_IN4: U6.8 (EXT_ADC1_IN4)
- new net ADC1_IN5: U6.7 (EXT_ADC1_IN5)
- new net GND: C18.2, C19.2, J1.2 (Pin_2), U6.18 (GND), U6.9 (GND)
- new net GPIO_A11: U6.4 (EXT_GPIO_PA11)
- new net GPIO_A12: U6.3 (EXT_GPIO_PA12)
- new net GPIO_PB3: U6.2 (EXT_GPIO_PB3)
- new net GPIO_PC15: U6.13 (EXT_GPIO_PC15)
- new net SYS_NRST: U6.10 (EXT_SYS_NRST)
- new net TIM17_CH1: U6.12 (EXT_TIM17_CH1)
- new net TIM17_CH1N: U6.11 (EXT_TIM17_CH1N)
- new net TIM1_CH1: U6.5 (EXT_TIM1_CH1)
- new net TIM1_CH1N: U6.6 (EXT_TIM1_CH1N)
- new net USART2_RX: U6.17 (EXT_USART2_RX)
- new net USART2_TX: U6.16 (EXT_USART2_TX)
- new net VDD: C18.1, C19.1, J1.1 (Pin_1), U6.1 (VDD)
