File: decoration.kicad_sch (KiCad schematic)
At the start: 9 parts, among them J12 Fuse holder or smth to hold t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

Commit message: Autosave
Connections:
- net UVLED3: now also R31.2
- net UVLED4: now also R32.2
Changed lines of the file:
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@@
 	(hierarchical_label "UVLED4"
 		(shape input)
-		(at 123.19 85.09 0)
+		(at 123.19 109.22 0)
 		(effects
 			(font
@@
 	(hierarchical_label "UVLED3"
 		(shape input)
-		(at 124.46 96.52 0)
+		(at 123.19 97.79 0)
 		(effects
 			(font

Commit message: Autosave
Parts:
- added J13, J14: Fuse holder or smth to hold tube, symbol Connector:Conn_01x02_Socket
Connections:
- no-connect marks 2 -> 6
Other:
- moved on the sheet: J12
Changed lines of the file:
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@@
 	)
 	(no_connect
-		(at 105.41 67.31)
+		(at 135.89 97.79)
 	)
 	(no_connect
-		(at 105.41 64.77)
+		(at 135.89 95.25)
+	)
+	(no_connect
+		(at 133.35 78.74)
+	)
+	(no_connect
+		(at 134.62 86.36)
+	)
+	(no_connect
+		(at 134.62 88.9)
+	)
+	(no_connect
+		(at 133.35 76.2)
 	)
 	(wire
@@
 	(symbol
 		(lib_id "Connector:Conn_01x02_Socket")
-		(at 110.49 64.77 0)
+		(at 138.43 76.2 0)
 		(unit 1)
 		(body_style 1)
@@
 		(fields_autoplaced yes)
 		(property "Reference" "J12"
-			(at 111.76 64.7699 0)
+			(at 139.7 76.1999 0)
 			(show_name no)
 			(do_not_autoplace no)
@@
 		)
 		(property "Value" "Fuse holder or smth to hold tube"
-			(at 111.76 67.3099 0)
+			(at 139.7 78.7399 0)
 			(show_name no)
 			(do_not_autoplace no)
@@
 		)
 		(property "Footprint" ""
-			(at 110.49 64.77 0)
+			(at 138.43 76.2 0)
 			(hide yes)
 			(show_name no)
@@
 		)
 		(property "Datasheet" ""
-			(at 110.49 64.77 0)
+			(at 138.43 76.2 0)
 			(hide yes)
 			(show_name no)
@@
 		)
 		(property "Description" "Generic connector, single row, 01x02, script generated"
-			(at 110.49 64.77 0)
+			(at 138.43 76.2 0)
 			(hide yes)
 			(show_name no)
@@
 	)
 	(symbol
+		(lib_id "Connector:Conn_01x02_Socket")
+		(at 140.97 95.25 0)
+		(unit 1)
+		(body_style 1)
+		(exclude_from_sim no)
+		(in_bom yes)
+		(on_board yes)
+		(in_pos_files yes)
+		(dnp no)
+		(fields_autoplaced yes)
+		(property "Reference" "J14"
+			(at 142.24 95.2499 0)
+			(show_name no)
+			(do_not_autoplace no)
+			(effects
+				(font
+					(size 1.27 1.27)
+				)
+				(justify left)
+			)
+		)
+		(property "Value" "Fuse holder or smth to hold tube"
+			(at 142.24 97.7899 0)
+			(show_name no)
+			(do_not_autoplace no)
+			(effects
+				(font
+					(size 1.27 1.27)
+				)
+				(justify left)
+			)
+		)
+		(property "Footprint" ""
+			(at 140.97 95.25 0)
+			(hide yes)
+			(show_name no)
+			(do_not_autoplace no)
+			(effects
+				(font
+					(size 1.27 1.27)
+				)
+			)
+		)
+		(property "Datasheet" ""
+			(at 140.97 95.25 0)
+			(hide yes)
+			(show_name no)
+			(do_not_autoplace no)
+			(effects
+				(font
+					(size 1.27 1.27)
+				)
+			)
+		)
+		(property "Description" "Generic connector, single row, 01x02, script generated"
+			(at 140.97 95.25 0)
+			(hide yes)
+			(show_name no)
+			(do_not_autoplace no)
+			(effects
+				(font
+					(size 1.27 1.27)
+				)
+			)
+		)
+		(pin "2"
+		)
+		(pin "1"
+		)
+		(instances
+			(project "WET_PCB_v2"
+				(path "/13451c35-1666-47d9-9525-8d8125ba1cf3/79e5e86e-dc26-4d0b-a087-2027a5880c08"
+					(reference "J14")
+					(unit 1)
+				)
+			)
+		)
+	)
+	(symbol
 		(lib_id "Device:R")
 		(at 119.38 77.47 90)
@@
 					(unit 1)
 				)
+			)
+		)
+	)
+	(symbol
+		(lib_id "Connector:Conn_01x02_Socket")
+		(at 139.7 86.36 0)
+		(unit 1)
+		(body_style 1)
+		(exclude_from_sim no)
+		(in_bom yes)
+		(on_board yes)
+		(in_pos_files yes)
+		(dnp no)
+		(fields_autoplaced yes)
+		(property "Reference" "J13"
+			(at 140.97 86.3599 0)
+			(show_name no)
+			(do_not_autoplace no)
+			(effects
+				(font
+					(size 1.27 1.27)
+				)
+				(justify left)
+			)
+		)
+		(property "Value" "Fuse holder or smth to hold tube"
+			(at 140.97 88.8999 0)
+			(show_name no)
+			(do_not_autoplace no)
+			(effects
+				(font
+					(size 1.27 1.27)
+				)
+				(justify left)
+			)
+		)
+		(property "Footprint" ""
+			(at 139.7 86.36 0)
+			(hide yes)
+			(show_name no)
+			(do_not_autoplace no)
+			(effects
+				(font
+					(size 1.27 1.27)
+				)
+			)
+		)
+		(property "Datasheet" ""
+			(at 139.7 86.36 0)
+			(hide yes)
+			(show_name no)
+			(do_not_autoplace no)
+			(effects
+				(font
+					(size 1.27 1.27)
+				)
+			)
+		)
+		(property "Description" "Generic connector, single row, 01x02, script generated"
+			(at 139.7 86.36 0)
+			(hide yes)
+			(show_name no)
+			(do_not_autoplace no)
+			(effects
+				(font
+					(size 1.27 1.27)
+				)
+			)
+		)
+		(pin "2"
+		)
+		(pin "1"
+		)
+		(instances
+			(project "WET_PCB_v2"
+				(path "/13451c35-1666-47d9-9525-8d8125ba1cf3/79e5e86e-dc26-4d0b-a087-2027a5880c08"
+					(reference "J13")
+					(unit 1)
+				)

Commit message: SCH Save: 1 files changed decoration.kicad_sch 90/0/9
Parts:
- added J15: Fuse holder or smth to hold tube, symbol Connector:Conn_01x02_Socket
Connections:
- no-connect marks 6 -> 8
Other:
- moved on the sheet: J14
Changed lines of the file:
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@@
 	)
 	(no_connect
-		(at 135.89 97.79)
+		(at 134.62 99.06)
 	)
 	(no_connect
-		(at 135.89 95.25)
+		(at 134.62 107.95)
+	)
+	(no_connect
+		(at 134.62 96.52)
+	)
+	(no_connect
+		(at 134.62 110.49)
 	)
 	(no_connect
@@
 	(symbol
 		(lib_id "Connector:Conn_01x02_Socket")
-		(at 140.97 95.25 0)
+		(at 139.7 96.52 0)
 		(unit 1)
 		(body_style 1)
@@
 		(fields_autoplaced yes)
 		(property "Reference" "J14"
-			(at 142.24 95.2499 0)
+			(at 140.97 96.5199 0)
 			(show_name no)
 			(do_not_autoplace no)
@@
 		)
 		(property "Value" "Fuse holder or smth to hold tube"
-			(at 142.24 97.7899 0)
+			(at 140.97 99.0599 0)
 			(show_name no)
 			(do_not_autoplace no)
@@
 		)
 		(property "Footprint" ""
-			(at 140.97 95.25 0)
+			(at 139.7 96.52 0)
 			(hide yes)
 			(show_name no)
@@
 		)
 		(property "Datasheet" ""
-			(at 140.97 95.25 0)
+			(at 139.7 96.52 0)
 			(hide yes)
 			(show_name no)
@@
 		)
 		(property "Description" "Generic connector, single row, 01x02, script generated"
-			(at 140.97 95.25 0)
+			(at 139.7 96.52 0)
 			(hide yes)
 			(show_name no)
@@
 					(unit 1)
 				)
+			)
+		)
+	)
+	(symbol
+		(lib_id "Connector:Conn_01x02_Socket")
+		(at 139.7 107.95 0)
+		(unit 1)
+		(body_style 1)
+		(exclude_from_sim no)
+		(in_bom yes)
+		(on_board yes)
+		(in_pos_files yes)
+		(dnp no)
+		(fields_autoplaced yes)
+		(property "Reference" "J15"
+			(at 140.97 107.9499 0)
+			(show_name no)
+			(do_not_autoplace no)
+			(effects
+				(font
+					(size 1.27 1.27)
+				)
+				(justify left)
+			)
+		)
+		(property "Value" "Fuse holder or smth to hold tube"
+			(at 140.97 110.4899 0)
+			(show_name no)
+			(do_not_autoplace no)
+			(effects
+				(font
+					(size 1.27 1.27)
+				)
+				(justify left)
+			)
+		)
+		(property "Footprint" ""
+			(at 139.7 107.95 0)
+			(hide yes)
+			(show_name no)
+			(do_not_autoplace no)
+			(effects
+				(font
+					(size 1.27 1.27)
+				)
+			)
+		)
+		(property "Datasheet" ""
+			(at 139.7 107.95 0)
+			(hide yes)
+			(show_name no)
+			(do_not_autoplace no)
+			(effects
+				(font
+					(size 1.27 1.27)
+				)
+			)
+		)
+		(property "Description" "Generic connector, single row, 01x02, script generated"
+			(at 139.7 107.95 0)
+			(hide yes)
+			(show_name no)
+			(do_not_autoplace no)
+			(effects
+				(font
+					(size 1.27 1.27)
+				)
+			)
+		)
+		(pin "2"
+		)
+		(pin "1"
+		)
+		(instances
+			(project "WET_PCB_v2"
+				(path "/13451c35-1666-47d9-9525-8d8125ba1cf3/79e5e86e-dc26-4d0b-a087-2027a5880c08"
+					(reference "J15")
+					(unit 1)
+				)
